File: Documentation/CMPET456_Lab7_Schematic.sch (EAGLE design)
At the start: 25 parts

Commit message: Updated PB VCC to be marked as +3.3VDC
Changed lines of the file:
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@@
 <part name="BLU_PB" library="SparkFun-Retired" deviceset="TAC_SWITCH" device="PTH"/>
 <part name="YEL_PB" library="SparkFun-Retired" deviceset="TAC_SWITCH" device="PTH"/>
-<part name="+3.3VDC" library="SparkFun-Aesthetics" deviceset="VCC" device="" value="VCC (5 VDC)"/>
+<part name="+3.3VDC" library="SparkFun-Aesthetics" deviceset="VCC" device="" value="VCC (+3.3 VDC)"/>
 <part name="GND1" library="SparkFun-Aesthetics" deviceset="GND" device=""/>
 <part name="R1" library="SparkFun-Passives" deviceset="RESISTOR" device="EZ"/>
